Commit message: add rectbot cv

File: src/rectbot_description/urdf/rectbot.urdf (robot description, URDF)
Before this commit: robot rectbot, 10 links, 9 joints
Joints:
- joint camera_joint: origin xyz=0.082529 -0.0026396 0.1145 rpy=0 0 0 -> xyz=0.12085 0.0175 0.09 rpy=0.0 0.0 0.0
- joint lidar_joint: origin xyz=-0.0068617 0 0.155 rpy=0 0 3.14 -> xyz=-0.0068617 0 0.103 rpy=0 0 3.14

Commit message: new BT

File: src/rectbot_description/urdf/rectbot.urdf (robot description, URDF)
Before this commit: robot rectbot, 10 links, 9 joints
Joints:
- joint lidar_joint: origin xyz=-0.0068617 0 0.103 rpy=0 0 3.14 -> xyz=-0.0068617 0 0.135 rpy=0 0 3.14
